Commit message: 1 joint fixed and rviz config is set for work

File: urdf/cart.urdf (robot description, URDF)
Before this commit: robot cart, 1 links, 0 joints
Links:
- removed link base
- added link forarm; visual box size=1 0.5 5
- added link shoulder; visual box size=1 10 0.5
Joints:
- added joint elbow: type fixed, parent shoulder, child forarm, origin xyz=0 0 0

Commit message: 2 links with continuous joint

File: urdf/cart.urdf (robot description, URDF)
Before this commit: robot cart, 2 links, 1 joints
Links:
- removed link forarm
- removed link shoulder
- added link base; visual cylinder length=1 radius=1
- added link rotor; visual box size=5 2 0.5
Joints:
- removed joint elbow
- added joint baseRotor: type continuous, parent base, child rotor, origin xyz=0 0 1
